File: tp8_DAC/tp8_ej2/TP8_ej2_Salomon/TP8_ej2_Salomon.kicad_sch (KiCad schematic)
At the start: 21 parts, among them J1 alimentacion, J2 alimentacion, J3 alimentacion, Q1 BC548, Q2 BC547, Q3 BC548

Commit message: update
Parts:
- J1: footprint TerminalBlock:TerminalBlock_bornier-2_P5.08mm -> TerminalBlock:TerminalBlock_MaiXu_MX126-5.0-02P_1x02_P5.00mm
- J2: value alimentacion -> input; footprint TerminalBlock:TerminalBlock_bornier-2_P5.08mm -> TerminalBlock:TerminalBlock_MaiXu_MX126-5.0-02P_1x02_P5.00mm
- J3: value alimentacion -> output; footprint TerminalBlock:TerminalBlock_bornier-2_P5.08mm -> TerminalBlock:TerminalBlock_MaiXu_MX126-5.0-02P_1x02_P5.00mm
- renumbered RB to RB1, Rs to Rs1
Connections:
- net at J3.1 (Pin_1): now also C5.2
- net at J1.1 (Pin_1): no longer C5.2

Commit message: update_schematics_ej2
Parts:
- added H1, H2, H3, H4: MountingHole_Pad, MountingHole:MountingHole_2.2mm_M2_Pad_Via, symbol Mechanical:MountingHole_Pad
- added TP1, TP2, TP3, TP4, TP5, TP6: TestPoint_Alt, TestPoint:TestPoint_Keystone_5000-5004_Miniature, symbol Connector:TestPoint_Alt
Connections:
- net at C2.1, Q1.3 (E), RE1.1: now also TP2.1
- net at C2.2, Q2.2 (B), R1.2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: now also TP3.1
- net at C1.2, Q1.2 (B), RB1.2: now also TP1.1
- net at C4.1, Q2.3 (E), RE2.1: now also TP4.1
- net +9V: now reaches J1.1 (Pin_1)
- net +9V: now also Q1.1 (C), Q3.1 (C), R1.1, R3.1, RB1.1, RC2.1
- net at C5.1, Q3.3 (E), RE3.1: now also TP6.1
- net at C3.2, Q3.2 (B), R3.2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: now also TP5.1
Other:
- moved on the sheet: J1
