File: tp8_DAC/tp8_ej1/TP8_ej1_Salomon.kicad_pcb (KiCad board)
At the start: 2 copper layers, 41.5 x 41.3 mm, 16 parts, among them Q1 BC548

Commit message: update_final
Parts:
- added H1: MountingHole_Pad, MountingHole:MountingHole_2.2mm_M2_Pad_Via, F.Cu at (2.48, 2.48)
- added H2: MountingHole_Pad, MountingHole:MountingHole_2.2mm_M2_Pad_Via, F.Cu at (2.48, 8.43)
- added H4: MountingHole_Pad, MountingHole:MountingHole_2.2mm_M2_Pad_Via, F.Cu at (2.48, 14.4)
- added TP1: TestPoint_Alt, Connector_Pin:Pin_D1.3mm_L11.0mm_LooseFit, F.Cu at (143.6, 70.0)
- added TP2: ~, Connector_Pin:Pin_D1.3mm_L11.0mm_LooseFit, F.Cu at (141.7, 91.4)
- renumbered input to J1, + to J2, output to J3
Connections:
- H3 pad 1: GND -> unconnected-(H3-Pad1)
Routing:
- net Net-(Q1-B): track 14.2 -> 33.7 mm
- net Net-(Q1-E): track 21.6 -> 25.8 mm
Other:
- board text added: "Salomon Franco"
- board text added: "TP8 - Ejercicio 1"
- board text added: "input"
- board text added: "output"
- board text removed: "Ejercicio 1 - TP8"
