File: tp8_DAC/tp8_ej1/TP8_ej1_Salomon.kicad_sch (KiCad schematic)
At the start: 11 parts, among them J1 Input_signal, J2 alimentacion, J3 output_signal, Q1 BC548

Commit message: update_final
Parts:
- added H2, H4: MountingHole_Pad, MountingHole:MountingHole_2.2mm_M2_Pad_Via, symbol Mechanical:MountingHole_Pad
- added TP1: TestPoint_Alt, Connector_Pin:Pin_D1.3mm_L11.0mm_LooseFit, symbol Connector:TestPoint_Alt
- added TP2: ~, Connector_Pin:Pin_D1.3mm_L11.0mm_LooseFit, symbol Connector:TestPoint_Alt
Connections:
- net at C1.2, Q1.2 (B), R3.2: now also TP1.1
- net at C2.1, Q1.3 (E), R4.1: now also TP2.1
