File: tp9_DAC/tp10_DAC.kicad_sch (KiCad schematic)
At the start: 35 parts, among them J2 BAT1, U1 NE555P, U2 NE555P

Commit message: entrega_tp10
Parts:
- J2: value BAT1 -> Bornera_2pos
- RL2: value 100 -> 100k
- TP1, TP2, TP3, TP4, TP5: now left out of the parts list
Changed lines of the file:
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@@
 			)
 		)
-		(property "Value" "100"
+		(property "Value" "100k"
 			(at 227.33 100.3299 0)
 			(effects
@@
 			)
 		)
-		(property "Value" "BAT1"
+		(property "Value" "Bornera_2pos"
 			(at 50.8 97.7899 0)
 			(effects
@@
 		(unit 1)
 		(exclude_from_sim no)
-		(in_bom yes)
+		(in_bom no)
 		(on_board yes)
 		(dnp no)
@@
 		(unit 1)
 		(exclude_from_sim no)
-		(in_bom yes)
+		(in_bom no)
 		(on_board yes)
 		(dnp no)
@@
 		(unit 1)
 		(exclude_from_sim no)
-		(in_bom yes)
+		(in_bom no)
 		(on_board yes)
 		(dnp no)
@@
 		(unit 1)
 		(exclude_from_sim no)
-		(in_bom yes)
+		(in_bom no)
 		(on_board yes)
 		(dnp no)
@@
 		(unit 1)
 		(exclude_from_sim no)
-		(in_bom yes)
-		(on_board yes)
-		(dnp no)
+		(in_bom no)
+		(on_board yes)
+		(dnp no)
