File: tp9_DAC/tp10_DAC.kicad_pcb (KiCad board)
At the start: 2 copper layers, 83.7 x 57.6 mm, 35 parts, among them J2 BAT1, U1 NE555P, U2 NE555P

Commit message: update_PCB
Parts:
- moved RL1 1.54 mm to (95.2, 70.5)
Routing:
- net +12V: track 172.1 -> 170.3 mm
- net Net-(U1-CV): track 11.2 -> 10.1 mm
- net Net-(U1-DIS): track 48.2 -> 47.1 mm

Commit message: retoques_cnc
Parts:
- moved TP4 1.36 mm to (125.7, 81.0)
- moved TP2 0.45 mm to (119.8, 89.7)
Changed lines of the file:
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@@
 	(footprint "TestPoint:TestPoint_THTPad_D1.0mm_Drill0.5mm"
 		(layer "F.Cu")
-		(at 120.3 89.7)
+		(at 119.85 89.74)
 		(descr "THT pad as test Point, diameter 1.0mm, hole diameter 0.5mm")
 		(tags "test point THT pad")
@@
 	(footprint "TestPoint:TestPoint_THTPad_D1.0mm_Drill0.5mm"
 		(layer "F.Cu")
-		(at 127 80.7)
+		(at 125.66 80.95)
 		(descr "THT pad as test Point, diameter 1.0mm, hole diameter 0.5mm")
 		(tags "test point THT pad")
@@
 		(start 92.75 58.65)
 		(end 87.9 63.5)
-		(width 1.27)
+		(width 1.524)
 		(layer "B.Cu")
 		(net 6)
@@
 		(start 107.42 81.965)
 		(end 107.42 81.72)
-		(width 1.016)
+		(width 1.524)
 		(layer "B.Cu")
 		(net 6)
@@
 		(start 99.7 58.65)
 		(end 92.75 58.65)
-		(width 1.27)
+		(width 1.524)
 		(layer "B.Cu")
 		(net 6)
@@
 		(start 87.9 73.76)
 		(end 92.74 78.6)
-		(width 1.27)
+		(width 1.524)
 		(layer "B.Cu")
 		(net 6)
@@
 		(start 104.3 78.6)
 		(end 94.93 78.6)
-		(width 1.016)
+		(width 1.27)
 		(layer "B.Cu")
 		(net 6)
@@
 		(start 92.74 78.6)
 		(end 94.93 78.6)
-		(width 1.27)
+		(width 1.524)
 		(layer "B.Cu")
 		(net 6)
@@
 		(start 87.9 63.5)
 		(end 87.9 73.76)
-		(width 1.27)
+		(width 1.524)
 		(layer "B.Cu")
 		(net 6)
@@
 		(start 107.42 81.72)
 		(end 104.3 78.6)
-		(width 1.016)
+		(width 1.27)
 		(layer "B.Cu")
 		(net 6)
@@
 		(start 134.6 90.4)
 		(end 127.25 90.4)
-		(width 1.524)
+		(width 2.159)
 		(layer "B.Cu")
 		(net 7)
@@
 		(start 134.6 90.4)
 		(end 147.3 90.4)
-		(width 1.524)
+		(width 2.159)
 		(layer "B.Cu")
 		(net 7)
@@
 		(start 127.25 90.4)
 		(end 126.6 89.75)
-		(width 1.524)
+		(width 2.159)
 		(layer "B.Cu")
 		(net 7)
@@
 	)
 	(segment
+		(start 119.51 90.49)
+		(end 119.51 90.08)
+		(width 2.159)
+		(layer "B.Cu")
+		(net 10)
+	)
+	(segment
 		(start 111.82 87.13)
 		(end 104.88 87.13)
@@
 		(start 84.77 85.57)
 		(end 88.3 89.1)
-		(width 1.7)
+		(width 2.159)
 		(layer "B.Cu")
 		(net 10)
@@
 		(start 88.3 89.1)
 		(end 99.51 89.1)
-		(width 1.7)
+		(width 2.159)
 		(layer "B.Cu")
 		(net 10)
@@
 	)
 	(segment
+		(start 119.51 90.08)
+		(end 119.85 89.74)
+		(width 2.159)
+		(layer "B.Cu")
+		(net 10)
+	)
+	(segment
 		(start 109.1 77)
 		(end 111.7 77)
@@
 		(start 100.9 90.49)
 		(end 113.6 90.49)
-		(width 1.7)
+		(width 2.159)
 		(layer "B.Cu")
 		(net 10)
@@
 		(start 113.6 90.49)
 		(end 119.51 90.49)
-		(width 1.7)
+		(width 2.159)
 		(layer "B.Cu")
 		(net 10)
@@
 		(start 84.75 78.62)
 		(end 84.77 78.6)
-		(width 1.7)
+		(width 2.159)
 		(layer "B.Cu")
 		(net 10)
@@
 	)
 	(segment
-		(start 119.51 90.49)
-		(end 120.3 89.7)
-		(width 1.7)
-		(layer "B.Cu")
-		(net 10)
-	)
-	(segment
 		(start 107.42 75.32)
 		(end 109.1 77)
@@
 		(start 99.51 89.1)
 		(end 100.9 90.49)
-		(width 1.7)
+		(width 2.159)
 		(layer "B.Cu")
 		(net 10)
@@
 		(start 84.77 78.6)
 		(end 84.77 85.57)
-		(width 1.7)
+		(width 2.159)
 		(layer "B.Cu")
 		(net 10)
@@
 		(start 139.29 83.69)
 		(end 139.29 82)
-		(width 1.27)
+		(width 1.524)
 		(layer "B.Cu")
 		(net 11)
 	)
 	(segment
-		(start 127 82.42)
-		(end 130.13 85.55)
-		(width 1.27)
+		(start 130.13 85.55)
+		(end 130.13 85.42)
+		(width 1.524)
 		(layer "B.Cu")
 		(net 11)
 	)
 	(segment
-		(start 127 80.7)
-		(end 127 82.42)
-		(width 1.27)
+		(start 130.13 85.42)
+		(end 125.66 80.95)
+		(width 1.524)
 		(layer "B.Cu")
 		(net 11)
@@
 		(start 130.13 85.55)
 		(end 137.43 85.55)
-		(width 1.27)
+		(width 1.524)
 		(layer "B.Cu")
 		(net 11)
@@
 		(start 137.43 85.55)
 		(end 139.29 83.69)
-		(width 1.27)
+		(width 1.524)
 		(layer "B.Cu")
 		(net 11)

Commit message: silkscreen
Parts:
- renumbered J2 to POWER
Other:
- board text added: "+"
- board text added: "TP1"
- board text added: "U1"
Changed lines of the file:
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@@
 			(at 0 -2.85 0)
 			(layer "F.SilkS")
+			(hide yes)
 			(effects
 				(font
@@
 		(tags "Resistor Axial_DIN0207 series Axial Horizontal pin pitch 10.16mm 0.25W = 1/4W length 6.3mm diameter 2.5mm")
 		(property "Reference" "RL1"
-			(at 5.08 -2.37 0)
+			(at 5.21 0.03 0)
 			(layer "F.SilkS")
 			(effects
@@
 		(descr "terminal block Metz Connect Type011_RT05502HBLC, 2 pins, pitch 5mm, size 10x10.5mm, drill diameter 1.4mm, pad diameter 2.8mm, https://americancableassemblies.com/content/metz/863188.PDF, script-generated using https://gitlab.com/kicad/libraries/kicad-footprint-generator/-/tree/master/scripts/TerminalBlock_MetzConnect")
 		(tags "THT terminal block Metz Connect Type011_RT05502HBLC pitch 5mm size 10x10.5mm drill 1.4mm pad 2.8mm")
-		(property "Reference" "J2"
-			(at 2.5 -7.62 90)
+		(property "Reference" "POWER"
+			(at 11.425 3.1275 270)
 			(layer "F.SilkS")
 			(effects
@@
 		(tags "C Radial series Radial pin pitch 2.00mm diameter 5mm height 11mm Non-Polar Electrolytic Capacitor")
 		(property "Reference" "C3"
-			(at 1 -3.75 90)
+			(at 1.12 -3.93 90)
 			(layer "F.SilkS")
 			(effects
@@
 			(at 0 -2.85 0)
 			(layer "F.SilkS")
+			(hide yes)
 			(effects
 				(font
@@
 			(at 0.85 -5.96 0)
 			(layer "F.SilkS")
+			(hide yes)
 			(effects
 				(font
@@
 		(tags "C Radial series Radial pin pitch 2.00mm diameter 5mm height 11mm Non-Polar Electrolytic Capacitor")
 		(property "Reference" "CV1"
-			(at 1 -3.75 0)
+			(at 5.4 0 90)
 			(layer "F.SilkS")
 			(effects
@@
 		(tags "test point THT pad")
 		(property "Reference" "TP2"
-			(at -2.1 1.8 0)
+			(at 0.43 2.01 0)
 			(layer "F.SilkS")
 			(effects
@@
 		(tags "Resistor Axial_DIN0207 series Axial Horizontal pin pitch 10.16mm 0.25W = 1/4W length 6.3mm diameter 2.5mm")
 		(property "Reference" "RA12"
-			(at 5.08 -2.37 0)
+			(at 5.29 -0.14 0)
 			(layer "F.SilkS")
 			(effects
@@
 		(tags "test point THT pad")
 		(property "Reference" "TP5"
-			(at 0 -1.448 0)
+			(at 0.05 2.4 0)
 			(layer "F.SilkS")
 			(effects
@@
 		(tags "test point THT pad")
 		(property "Reference" "TP3"
-			(at -1.6 1.75 0)
+			(at -0.13 2 0)
 			(layer "F.SilkS")
 			(effects
@@
 		(tags "Resistor Axial_DIN0207 series Axial Horizontal pin pitch 10.16mm 0.25W = 1/4W length 6.3mm diameter 2.5mm")
 		(property "Reference" "RB1"
-			(at 5.08 -2.37 0)
+			(at 5.11 -0.06 0)
 			(layer "F.SilkS")
 			(effects
@@
 		(tags "Resistor Axial_DIN0207 series Axial Horizontal pin pitch 10.16mm 0.25W = 1/4W length 6.3mm diameter 2.5mm")
 		(property "Reference" "RA11"
-			(at 5.08 -2.37 90)
+			(at 5.11 0.04 90)
 			(layer "F.SilkS")
 			(effects
@@
 		(tags "C Radial series Radial pin pitch 2.00mm diameter 5mm height 11mm Non-Polar Electrolytic Capacitor")
 		(property "Reference" "CV2"
-			(at 1 -3.75 90)
+			(at 4.95 0.11 180)
 			(layer "F.SilkS")
 			(effects
@@
 		(tags "C Radial series Radial pin pitch 2.00mm diameter 5mm height 11mm Non-Polar Electrolytic Capacitor")
 		(property "Reference" "C6"
-			(at 0.95 2 0)
+			(at 0.86 3.77 0)
 			(layer "F.SilkS")
 			(effects
@@
 		(tags "C Radial series Radial pin pitch 2.00mm diameter 5mm height 11mm Non-Polar Electrolytic Capacitor")
 		(property "Reference" "C5"
-			(at 1 -3.75 90)
+			(at 0.86 -3.87 90)
 			(layer "F.SilkS")
 			(effects
@@
 			(at 0 -2.85 0)
 			(layer "F.SilkS")
+			(hide yes)
 			(effects
 				(font
@@
 			(at 0.1 -0.4 0)
 			(layer "F.SilkS")
+			(hide yes)
 			(effects
 				(font
@@
 		(tags "C Radial series Radial pin pitch 2.00mm diameter 5mm height 11mm Non-Polar Electrolytic Capacitor")
 		(property "Reference" "C2"
-			(at 1 -3.75 0)
+			(at 4.82 0.01 90)
 			(layer "F.SilkS")
 			(effects
@@
 		(tags "test point THT pad")
 		(property "Reference" "TP4"
-			(at 0.15 2.25 0)
+			(at 0.06 -2.05 0)
 			(layer "F.SilkS")
 			(effects
@@
 			(at 2.875 -0.1 90)
 			(layer "F.SilkS")
+			(hide yes)
 			(effects
 				(font
@@
 		(tags "C Radial series Radial pin pitch 2.00mm diameter 5mm height 11mm Non-Polar Electrolytic Capacitor")
 		(property "Reference" "C7"
-			(at 1 -2.1844 0)
+			(at 1.04 -3.83 0)
 			(layer "F.SilkS")
 			(effects
@@
 		(tags "C Radial series Radial pin pitch 2.00mm diameter 5mm height 11mm Non-Polar Electrolytic Capacitor")
 		(property "Reference" "C1"
-			(at 1 -3.75 0)
+			(at 4.64 0.16 90)
 			(layer "F.SilkS")
 			(effects
@@
 		(tags "C Radial series Radial pin pitch 2.00mm diameter 5mm height 11mm Non-Polar Electrolytic Capacitor")
 		(property "Reference" "C11"
-			(at 1 -3.75 0)
+			(at 0.87 -3.5 0)
 			(layer "F.SilkS")
 			(effects
@@
 		(tags "C Radial series Radial pin pitch 2.00mm diameter 5mm height 11mm Non-Polar Electrolytic Capacitor")
 		(property "Reference" "C12"
-			(at 1 -3.75 0)
+			(at 0.97 3.87 0)
 			(layer "F.SilkS")
 			(effects
@@
 		(tags "THT DIP DIL PDIP 2.54mm 7.62mm 300mil")
 		(property "Reference" "U2"
-			(at 3.81 -2.33 90)
+			(at 3.71 3.87 0)
 			(layer "F.SilkS")
 			(effects
@@
 		(tags "Resistor Axial_DIN0207 series Axial Horizontal pin pitch 10.16mm 0.25W = 1/4W length 6.3mm diameter 2.5mm")
 		(property "Reference" "RL2"
-			(at 5.08 -2.37 0)
+			(at 5.14 -0.06 0)
 			(layer "F.SilkS")
 			(effects
@@
 		(layer "Edge.Cuts")
 	)
+	(gr_text "TP1\n"
+		(at 119.82 78.76 0)
+		(layer "F.SilkS")
+		(effects
+			(font
+				(size 1 1)
+				(thickness 0.15)
+			)
+		)
+	)
+	(gr_text "U1\n\n"
+		(at 105.84 78.52 0)
+		(layer "F.SilkS")
+		(effects
+			(font
+				(size 1 1)
+				(thickness 0.15)
+			)
+		)
+	)
+	(gr_text "+\n"
+		(at 163.49 88.4 0)
+		(layer "F.SilkS")
+		(effects
+			(font
+				(size 1.5 1.5)
+				(thickness 0.3)
+				(bold yes)
+			)
+			(justify left bottom mirror)
+		)
+	)
 	(segment
