File: proyecto_danna/design_heart/design_heart.kicad_sch (KiCad schematic)
At the start: 24 parts, among them Q1 BC548, U1 LM358

Commit message: update_heart
Parts:
- removed D1, D2, D6: LED, LED_THT:LED_D5.0mm_IRGrey, symbol Device:LED
- removed unit 2 of U1
- removed unit 1 of U1
- added D13, D14, D15: LED, LED_THT:LED_D5.0mm_IRGrey, symbol Device:LED
- added U2: LM358, Package_DIP:DIP-8_W7.62mm_Socket, symbol Amplifier_Operational:LM358
Connections:
- net +12V: no longer U1.8 (V+)
- net GND: now also D13.1 (K), D14.1 (K), D15.1 (K), U2.4 (V-); no longer D10.1 (K), D11.1 (K), D12.1 (K), D3.1 (K), D4.1 (K), D5.1 (K)
- net breath: now also U2.1
- net at D10.2 (A), D11.2 (A), D12.2 (A)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: no longer D7.2 (A), D8.2 (A), D9.2 (A)
- net at C1.2, R2.1: now also U2.2 (-)
- net at R3.1, R4.1: now also U2.5 (+)
- net at R2.2, R4.2: now also U2.7
- net at R5.2, R6.1: now also U2.3 (+), U2.6 (-)
- new net: D12.1 (K), D9.2 (A)
- new net: D14.2 (A), D4.1 (K)
- new net: D15.2 (A), D5.1 (K)
- new net: D13.2 (A), D3.1 (K)
- new net: D11.1 (K), D8.2 (A)
- new net: D10.1 (K), D7.2 (A)
- new net: U1.8 (V+), U2.8 (V+)
Other:
- moved on the sheet: D10, D11, D12, D3, D4, D7, D8, D9

Commit message: update_heart
Parts:
- added D1: LED, LED_THT:LED_D5.0mm_IRGrey, symbol Device:LED
- added J1: Screw_Terminal_01x02, TerminalBlock_MetzConnect:TerminalBlock_MetzConnect_Type059_RT06302HBWC_1x02_P3.50mm_Horizontal, symbol Connector:Screw_Terminal_01x02
- added SW1: SW_Nidec_CAS-120A1, Button_Switch_SMD:Nidec_Copal_CAS-120A, symbol Switch:SW_Nidec_CAS-120A1
Connections:
- net +12V: now also U1.8 (V+), U2.8 (V+), SW1.2 (B)
- net GND: now also D1.1 (K), J1.2 (Pin_2)
- new net +12V_pre: D1.2 (A), J1.1 (Pin_1), SW1.3 (A)

Commit message: update_heart
Parts:
- added R8: 220, Resistor_THT:R_Axial_DIN0204_L3.6mm_D1.6mm_P7.62mm_Horizontal, symbol Device:R_Small
Connections:
- net +12V_pre: now also R8.1; no longer D1.2 (A)
- new net: D1.2 (A), R8.2
Other:
- moved on the sheet: D1
Changed lines of the file:
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@@
 	(wire
 		(pts
-			(xy 91.44 46.99) (xy 91.44 48.26)
+			(xy 91.44 54.61) (xy 91.44 55.88)
 		)
 		(stroke
@@
 	(wire
 		(pts
+			(xy 91.44 40.64) (xy 91.44 39.37)
+		)
+		(stroke
+			(width 0)
+			(type default)
+		)
+	)
+	(wire
+		(pts
 			(xy 106.68 105.41) (xy 106.68 107.95)
 		)
@@
 	(wire
 		(pts
+			(xy 91.44 46.99) (xy 91.44 45.72)
+		)
+		(stroke
+			(width 0)
+			(type default)
+		)
+	)
+	(wire
+		(pts
 			(xy 203.2 102.87) (xy 203.2 100.33)
 		)
@@
 	(symbol
 		(lib_id "power:GND")
-		(at 91.44 48.26 0)
+		(at 91.44 55.88 0)
 		(unit 1)
 		(exclude_from_sim no)
@@
 		(fields_autoplaced yes)
 		(property "Reference" "#PWR010"
-			(at 91.44 54.61 0)
+			(at 91.44 62.23 0)
 			(effects
 				(font
@@
 		)
 		(property "Value" "GND"
-			(at 91.44 53.34 0)
+			(at 91.44 60.96 0)
 			(effects
 				(font
@@
 		)
 		(property "Footprint" ""
-			(at 91.44 48.26 0)
+			(at 91.44 55.88 0)
 			(effects
 				(font
@@
 		)
 		(property "Datasheet" ""
-			(at 91.44 48.26 0)
+			(at 91.44 55.88 0)
 			(effects
 				(font
@@
 		)
 		(property "Description" "Power symbol creates a global label with name \"GND\" , ground"
-			(at 91.44 48.26 0)
+			(at 91.44 55.88 0)
 			(effects
 				(font
@@
 	)
 	(symbol
+		(lib_id "Device:R_Small")
+		(at 91.44 43.18 0)
+		(unit 1)
+		(exclude_from_sim no)
+		(in_bom yes)
+		(on_board yes)
+		(dnp no)
+		(fields_autoplaced yes)
+		(property "Reference" "R8"
+			(at 93.98 41.9099 0)
+			(effects
+				(font
+					(size 1.016 1.016)
+				)
+				(justify left)
+			)
+		)
+		(property "Value" "220"
+			(at 93.98 44.4499 0)
+			(effects
+				(font
+					(size 1.27 1.27)
+				)
+				(justify left)
+			)
+		)
+		(property "Footprint" "Resistor_THT:R_Axial_DIN0204_L3.6mm_D1.6mm_P7.62mm_Horizontal"
+			(at 91.44 43.18 0)
+			(effects
+				(font
+					(size 1.27 1.27)
+				)
+				(hide yes)
+			)
+		)
+		(property "Datasheet" "~"
+			(at 91.44 43.18 0)
+			(effects
+				(font
+					(size 1.27 1.27)
+				)
+				(hide yes)
+			)
+		)
+		(property "Description" "Resistor, small symbol"
+			(at 91.44 43.18 0)
+			(effects
+				(font
+					(size 1.27 1.27)
+				)
+				(hide yes)
+			)
+		)
+		(pin "1"
+		)
+		(pin "2"
+		)
+		(instances
+			(project "design_heart"
+				(path "/351bad0a-1beb-4827-907f-145a07d8f769"
+					(reference "R8")
+					(unit 1)
+				)
+			)
+		)
+	)
+	(symbol
 		(lib_id "Device:LED")
-		(at 91.44 43.18 90)
+		(at 91.44 50.8 90)
 		(unit 1)
 		(exclude_from_sim no)
@@
 		(dnp no)
 		(property "Reference" "D1"
-			(at 92.71 43.688 90)
+			(at 92.71 51.308 90)
 			(effects
 				(font
@@
 		)
 		(property "Value" "LED"
-			(at 92.71 42.164 90)
+			(at 92.71 49.784 90)
 			(effects
 				(font
@@
 		)
 		(property "Footprint" "LED_THT:LED_D5.0mm_IRGrey"
-			(at 91.44 43.18 0)
+			(at 91.44 50.8 0)
 			(effects
 				(font
@@
 		)
 		(property "Datasheet" "~"
-			(at 91.44 43.18 0)
+			(at 91.44 50.8 0)
 			(effects
 				(font
@@
 		)
 		(property "Description" "Light emitting diode"
-			(at 91.44 43.18 0)
+			(at 91.44 50.8 0)
 			(effects
 				(font
@@
 		)
 		(property "Sim.Pins" "1=K 2=A"
-			(at 91.44 43.18 0)
+			(at 91.44 50.8 0)
 			(effects
 				(font

Commit message: update_pcb_puentes
Parts:
- removed Q1: BC548, Package_TO_SOT_THT:TO-92_Inline, symbol Transistor_BJT:BC548
- removed RV1: 50k, Potentiometer_THT:Potentiometer_ACP_CA9-V10_Vertical_Hole, symbol Device:R_Potentiometer
- removed RV2: 1k, Potentiometer_THT:Potentiometer_ACP_CA9-V10_Vertical_Hole, symbol Device:R_Potentiometer
- removed SW1: SW_Nidec_CAS-120A1, Button_Switch_SMD:Nidec_Copal_CAS-120A, symbol Switch:SW_Nidec_CAS-120A1
- added Q2: BC548, Package_TO_SOT_THT:TO-92_Inline_Wide, symbol Transistor_BJT:BC548
- added RV3: 50k, Potentiometer_THT:Potentiometer_ACP_CA9-V10_Vertical, symbol Device:R_Potentiometer
- added RV4: 1k, Potentiometer_THT:Potentiometer_ACP_CA9-V10_Vertical, symbol Device:R_Potentiometer
- added S1: TL2230OAF140, TL2230OAF140:SW_TL2230OAF140, symbol TL2230OAF140:TL2230OAF140
Connections:
- net +12V: now also Q2.1 (C), S1.2
- net +12V_pre: now also S1.1
- net breath: now also Q2.2 (B), RV3.2, RV3.3
- net at R1.1, R7.1: now also RV4.3
- net at R3.2: now also RV3.1
- new net: Q2.3 (E), RV4.1, RV4.2
Other:
- moved on the sheet: D1, J1, R8
